File: pcb/LuMo.kicad_pcb (KiCad board)
At the start: 2 copper layers, 141 x 132 mm, 78 parts, among them J1 JST_02, J2 Display, J3 JST_02, J4 PINHD_1x2_Female, J5 Display, SW1 SW_Push, SW10 SW_Push, SW11 SW_Push, SW12 SW_Push, SW13 SW_Push, SW14 SW_Push, SW15 SW_Push, SW16 SW_Push, SW17 SW_Push, SW18 SW_Push, SW19 SW_Push, SW2 SW_Push, SW20 SW_Push, SW21 SW_Push, SW22 SW_Push, SW23 SW_Push, SW24 SW_Push, SW25 SW_Push, SW26 SW_Push, SW27 SW_Push, SW28 SW_Push, SW29 SW_Push, SW3 SW_Push, SW30 SW_Push, SW31 SW_Push, SW32 SW_Push, SW33 Reset, SW4 SW_Push, SW5 SW_Push, SW6 SW_Push, SW7 SW_Push, SW8 SW_Push, SW9 SW_Push, U1 ProMicro

Commit message: add first version of PCB
Parts:
- removed H5: MountingHole_M3_3.2mm_Pad, PCM_SL_Mechanical:MountingHole_3.2mm_Pad
- moved SW33 4.90 mm to (82.1, 25.4)
- moved D32 4.44 mm to (158.0, 145.2)
- moved SWI1 4.00 mm to (94.6, 27.9)
- moved D31 3.64 mm to (143.5, 140.5)
- moved D19 3.49 mm to (67.3, 105.3)
- moved D26 3.49 mm to (67.3, 124.3)
- moved D8 3.49 mm to (86.3, 78.6)
- moved D2 3.49 mm to (86.3, 59.6)
- moved D12 3.49 mm to (67.3, 86.2)
- moved D15 3.49 mm to (86.3, 97.7)
- moved D22 3.49 mm to (86.3, 116.7)
- moved D5 3.49 mm to (67.3, 67.2)
- moved D13 3.49 mm to (48.2, 91.0)
- moved D20 3.49 mm to (48.2, 110.1)
- moved D27 3.49 mm to (48.5, 129.1)
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Routing:
- net Row1: track 177.8 -> 166.6 mm, vias 4 -> 0
- net GND: track 180.9 -> 171.4 mm
- net Row2: track 218.7 -> 209.4 mm
- net Row4: track 235.3 -> 227.4 mm
- net Row5: track 219.8 -> 212.4 mm
- net Net-(D13-A): track 11.5 -> 6.27 mm
- net RST: track 48.5 -> 43.5 mm
- net Row3: track 218.0 -> 213.8 mm
- net Net-(D32-A): track 11.6 -> 15.5 mm, vias 0 -> 1
- net SCK: track 44.9 -> 42.0 mm
- net Net-(D5-A): track 12.7 -> 10.1 mm
- net Net-(D27-A): track 11.7 -> 9.77 mm
- net Net-(D30-A): track 11.6 -> 10.0 mm
- net Net-(D28-A): track 11.6 -> 10.0 mm
- net Net-(D29-A): track 11.6 -> 10.0 mm
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Other:
- outline, holes or cut-outs redrawn

Commit message: update kicad project
Parts:
- removed the J3 at (98.8, 36.0)
- J1: value JST_02 -> JST 1.25; footprint Connector_JST:JST_ACH_BM02B-ACHSS-GAN-ETF_1x02-1MP_P1.20mm_Vertical -> Connector_PinHeader_1.27mm:PinHeader_1x02_P1.27mm_Vertical
- J4: value PINHD_1x2_Female -> Magnetic Port
- moved J1 3.68 mm to (95.2, 35.4), turned to 0 degrees
- moved J4 0.39 mm to (164.5, 54.1)
- renumbered J5 to J2, J2 to J3
Connections:
- J1 pad 1: Net-(SWI1-A) -> VBAT
- SWI1 pad 1: Net-(SWI1-A) -> VBAT
- SWI1 pad 2: VBAT -> B+
- U1 pad 0: unconnected-(U1-B--Pad0) -> GND
- U1 pad 25: VBAT -> B+
- U1 pad 3: GND -> unconnected-(U1-GND-Pad3)
- U1 pad 4: GND -> unconnected-(U1-GND-Pad4)
Routing:
- net B+: track 0.00 -> 60.6 mm
- net VBAT: track 143.3 -> 85.0 mm, vias 2 -> 0
- net Net-(SWI1-A): track 14.9 -> 0.00 mm, vias 1 -> 0
- net GND: track 171.4 -> 183.9 mm, vias 3 -> 0
- net Col5: track 268.3 -> 267.8 mm, vias 7 -> 5
- net CS: track 58.9 -> 59.2 mm, vias 0 -> 2
