File: pcb/LuMo.kicad_sch (KiCad schematic)
At the start: 78 parts, among them J1 JST_02, J2 Display, J3 JST_02, J4 PINHD_1x2_Female, J5 Display, SW1 SW_Push, SW10 SW_Push, SW11 SW_Push, SW12 SW_Push, SW13 SW_Push, SW14 SW_Push, SW15 SW_Push, SW16 SW_Push, SW17 SW_Push, SW18 SW_Push, SW19 SW_Push, SW2 SW_Push, SW20 SW_Push, SW21 SW_Push, SW22 SW_Push, SW23 SW_Push, SW24 SW_Push, SW25 SW_Push, SW26 SW_Push, SW27 SW_Push, SW28 SW_Push, SW29 SW_Push, SW3 SW_Push, SW30 SW_Push, SW31 SW_Push, SW32 SW_Push, SW33 Reset, SW4 SW_Push, SW5 SW_Push, SW6 SW_Push, SW7 SW_Push, SW8 SW_Push, SW9 SW_Push, U1 ProMicro

Commit message: add first version of PCB
Changed lines of the file:
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@@
 	(wire
 		(pts
-			(xy 25.4 168.91) (xy 25.4 165.1)
+			(xy 30.48 166.37) (xy 30.48 165.1)
 		)
 		(stroke
@@
 	(wire
 		(pts
-			(xy 25.4 165.1) (xy 36.83 165.1)
+			(xy 30.48 165.1) (xy 36.83 165.1)
 		)
 		(stroke
@@
 	(symbol
 		(lib_id "tmk:GND")
-		(at 25.4 168.91 0)
+		(at 30.48 166.37 0)
 		(unit 1)
 		(exclude_from_sim no)
@@
 		(fields_autoplaced yes)
 		(property "Reference" "#PWR08"
-			(at 25.4 167.64 0)
+			(at 30.48 165.1 0)
 			(effects
 				(font
@@
 		)
 		(property "Value" "GND"
-			(at 25.4 167.64 0)
+			(at 30.48 165.1 0)
 			(effects
 				(font
@@
 		)
 		(property "Footprint" ""
-			(at 25.4 168.91 0)
+			(at 30.48 166.37 0)
 			(effects
 				(font
@@
 		)
 		(property "Datasheet" ""
-			(at 25.4 168.91 0)
+			(at 30.48 166.37 0)
 			(effects
 				(font
@@
 		)
 		(property "Description" ""
-			(at 25.4 168.91 0)
+			(at 30.48 166.37 0)
 			(effects
 				(font

Commit message: update kicad project
Parts:
- removed J1, J3: JST_02, Connector_JST:JST_ACH_BM02B-ACHSS-GAN-ETF_1x02-1MP_P1.20mm_Vertical, symbol PCM_SL_Connectors:JST_02
- added J1: JST 1.25, Connector_PinHeader_1.27mm:PinHeader_1x02_P1.27mm_Vertical, symbol PCM_SL_Pin_Headers:PINHD_1x2_Female
- J4: value PINHD_1x2_Female -> Magnetic Port
- renumbered J5 to J2, J2 to J3
Connections:
- net GND: now also U1.0 (B-), J1.2; no longer U1.3 (GND), U1.4 (GND)
- net VBAT: now also SWI1.1 (A), J1.1; no longer SWI1.2 (B), U1.25 (B+)
- new net B+: SWI1.2 (B), U1.25 (B+)
- no-connect marks 12 -> 13
Other:
- moved on the sheet: H1, H2, H3, H4, H5, H6, J2, J3, J4, SW33, SWI1
