File: pcb/LuMo_bottom.kicad_pcb (KiCad board)
At the start: 2 copper layers, 141 x 132 mm, 5 parts

Commit message: update kicad project
Changed lines of the file:
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@@
 			(at 0 0)
 			(size 6 6)
-			(drill 4.1)
+			(drill 3)
 			(layers "*.Cu" "*.Mask")
 			(remove_unused_layers no)
@@
 			(at 0 0)
 			(size 6 6)
-			(drill 4.1)
+			(drill 3)
 			(layers "*.Cu" "*.Mask")
 			(remove_unused_layers no)
@@
 			(at 0 0)
 			(size 6 6)
-			(drill 4.1)
+			(drill 3)
 			(layers "*.Cu" "*.Mask")
 			(remove_unused_layers no)
@@
 			(at 0 0)
 			(size 6 6)
-			(drill 4.1)
+			(drill 3)
 			(layers "*.Cu" "*.Mask")
 			(remove_unused_layers no)
@@
 			(at 0 0)
 			(size 6 6)
-			(drill 4.1)
-			(layers "*.Cu" "*.Mask")
-			(remove_unused_layers no)
+			(drill 3)
+			(layers "*.Cu" "*.Mask")
+			(remove_unused_layers no)
